File: MeshHat.kicad_pcb (KiCad board)
At the start: 2 copper layers, 65 x 56.5 mm, 26 parts, among them J1 RPi_GPIO, U5 RP2040, U6 W25Q128JVS, U7 E22-900M30S, Y1 ABM8-272-T3

Commit message: WIP
Parts:
- removed C1: 0U1, Capacitor_SMD:C_0603_1608Metric
- removed the J1 at (184.6, 54.3)
- removed the R1 at (94.2, 42.5)
- removed the R2 at (94.2, 45.0)
- removed R4: 1K, Resistor_SMD:R_0603_1608Metric
- removed U5: RP2040, Package_DFN_QFN:QFN-56-1EP_7x7mm_P0.4mm_EP3.2x3.2mm
- removed U6: W25Q128JVS, Package_SO:SOIC-8_5.3x5.3mm_P1.27mm
- removed U7: E22-900M30S, E22P:XCVR_E22-900M30S
- added C15: 0.1uF, Capacitor_SMD:C_0201_0603Metric, B.Cu at (194.1, 93.9)
- added C16: 26pF, Capacitor_SMD:C_0402_1005Metric, F.Cu at (197.2, 105.6)
- added D1: LED, LED_SMD:LED_0603_1608Metric, F.Cu at (200.4, 90.7)
- added J1: RPi_GPIO, RPi_HAT:RPI_Hat_B+, F.Cu at (204.5, 63.0)
- added J1: USB_A, Kevin_Lutzer_Lbr:USB3_A_Plug_Wuerth_629004113921_Horizontal, F.Cu at (82.2, 40.0)
- added R1: 2K2, Resistor_SMD:R_0603_1608Metric, F.Cu at (173.4, 117.3)
- added R1: 220, Resistor_SMD:R_0402_1005Metric, F.Cu at (198.6, 89.9)
- added R2: 2K2, Resistor_SMD:R_0603_1608Metric, F.Cu at (173.4, 119.8)
- added R2: 10k, Resistor_SMD:R_0402_1005Metric, F.Cu at (188.7, 94.0)
- added U2: W25Q32JVZP, Package_SON:WSON-8-1EP_6x5mm_P1.27mm_EP3.4x4.3mm, F.Cu at (191.8, 90.1)
- added U3: RP2040, Kevin_Lutzer_Lbr:RP2040-QFN-56, F.Cu at (194.9, 97.7)
- C10, C11, C8, C9: value 0U1 -> 0.1uF; footprint Capacitor_SMD:C_0603_1608Metric -> Capacitor_SMD:C_0201_0603Metric; moved to B.Cu
- C12: value 0U1 -> 26pF; footprint Capacitor_SMD:C_0603_1608Metric -> Capacitor_SMD:C_0402_1005Metric
- C13, C5: value 0U1 -> 0.1uF; footprint Capacitor_SMD:C_0603_1608Metric -> Capacitor_SMD:C_0201_0603Metric
- C14: value 0U1 -> 1uF; footprint Capacitor_SMD:C_0603_1608Metric -> Capacitor_SMD:C_0402_1005Metric
- C2: value 15P -> 1uF; footprint Capacitor_SMD:C_0603_1608Metric -> Capacitor_SMD:C_0402_1005Metric; moved to B.Cu
- C3: value 15P -> 0.1uF; footprint Capacitor_SMD:C_0603_1608Metric -> Capacitor_SMD:C_0201_0603Metric
- C4, C7: value 1U -> 0.1uF; footprint Capacitor_SMD:C_0603_1608Metric -> Capacitor_SMD:C_0201_0603Metric
- C6: value 0U1 -> 1uF; footprint Capacitor_SMD:C_0603_1608Metric -> Capacitor_SMD:C_0402_1005Metric; moved to B.Cu
- R3: value 1K -> 1k; footprint Resistor_SMD:R_0603_1608Metric -> Resistor_SMD:R_0402_1005Metric
- R5: value 27.4 -> 10k; footprint Resistor_SMD:R_0603_1608Metric -> Resistor_SMD:R_0402_1005Metric
- R6: footprint Resistor_SMD:R_0603_1608Metric -> Resistor_SMD:R_0201_0603Metric
- R7: value 10K -> 27.4; footprint Resistor_SMD:R_0603_1608Metric -> Resistor_SMD:R_0201_0603Metric
- Y1: value ABM8-272-T3 -> Crystal_GND24; footprint Crystal:Crystal_SMD_Abracon_ABM8G-4Pin_3.2x2.5mm -> Crystal:Crystal_SMD_2520-4Pin_2.5x2.0mm
- moved C3 128.4 mm to (199.5, 94.8), turned to -90 degrees
- moved C2 127.5 mm to (197.3, 95.2), turned to 180 degrees
- moved C8 126.0 mm to (196.1, 100.2), turned to 180 degrees
- moved R3 125.0 mm to (197.2, 103.6), turned to 90 degrees
- moved R5 124.2 mm to (200.1, 101.4), turned to 180 degrees
- moved C13 123.2 mm to (199.5, 98.4), turned to -90 degrees
- moved C9 123.2 mm to (197.1, 94.2), turned to 180 degrees
- moved C7 123.0 mm to (197.9, 93.1), turned to 180 degrees
- moved C4 120.3 mm to (190.3, 98.4), turned to -90 degrees
- moved C12 119.9 mm to (192.6, 103.6), turned to -90 degrees
- moved C11 118.7 mm to (194.1, 94.8)
- moved C5 117.7 mm to (190.2, 94.2), turned to -90 degrees
- moved C10 116.9 mm to (193.6, 88.6), turned to 90 degrees
- moved R6 115.6 mm to (195.9, 92.0), turned to 90 degrees
- moved R7 115.5 mm to (196.7, 92.0), turned to 90 degrees
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Connections:
- C10 pad 1: +3.3V -> GND
- C10 pad 2: GND -> +3V3
- C11 pad 1: +3.3V -> GND
- C11 pad 2: GND -> +1V1
- C12 pad 1: +3.3V -> GND
- C12 pad 2: GND -> /X_IN
- C13 pad 1: +3.3V -> GND
- C13 pad 2: GND -> +3V3
- C14 pad 1: +3.3V -> GND
- C14 pad 2: GND -> +3V3
- C2 pad 2: Net-(C2-Pad2) -> +1V1
- C3 pad 1: Net-(C3-Pad1) -> GND
- C3 pad 2: GND -> +3V3
- C4 pad 1: +1V1 -> GND
- C4 pad 2: GND -> +3V3
- C5 pad 1: +1V1 -> GND
- C5 pad 2: GND -> +3V3
- C6 pad 1: +1V1 -> GND
- C6 pad 2: GND -> +3V3
- C7 pad 1: +3.3V -> GND
- C7 pad 2: GND -> +3V3
- C8 pad 1: +3.3V -> GND
- C8 pad 2: GND -> +3V3
- C9 pad 1: +3.3V -> GND
- C9 pad 2: GND -> +1V1
- R3 pad 1: R_USB_BOOT -> Net-(C16-Pad2)
- R3 pad 2: /MeshRF/~{F_SS} -> /X_OUT
- R5 pad 1: /MeshRF/R_USB_DM -> +3V3
- R5 pad 2: Net-(U5-USB_DM) -> /RESET
- R6 pad 1: /MeshRF/R_USB_DP -> /USBR_+
- R6 pad 2: Net-(U5-USB_DP) -> /USB_+
- R7 pad 1: +3.3V -> /USBR_-
- R7 pad 2: R_RUN -> /USB_-
- Y1 pad 1: Net-(C3-Pad1) -> /X_IN
- Y1 pad 3: Net-(C2-Pad2) -> Net-(C16-Pad2)
Routing:
- net /QSPI_CS: track 0.00 -> 25.5 mm, vias 0 -> 2
- net GND: track 0.00 -> 21.5 mm, vias 0 -> 18
- net +3V3: track 0.00 -> 18.7 mm, vias 0 -> 10
- net +1V1: track 0.00 -> 16.8 mm, vias 0 -> 2
- net /QSPI_SD1: track 0.00 -> 9.55 mm, vias 0 -> 2
- net /RESET: track 0.00 -> 8.92 mm
- net /QSPI_SD2: track 0.00 -> 7.61 mm
- net /X_IN: track 0.00 -> 6.93 mm
- net /LED: track 0.00 -> 6.20 mm
- net /QSPI_SD3: track 0.00 -> 5.54 mm
- net /QSPI_SCLK: track 0.00 -> 4.23 mm
- net /X_OUT: track 0.00 -> 3.67 mm
- net /USB_-: track 0.00 -> 3.26 mm
- net Net-(C16-Pad2): track 0.00 -> 2.69 mm
- net /QSPI_SD0: track 0.00 -> 2.67 mm
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Other:
- copper layers 2 -> 4
- board text added: "Layout on 0.1mm Traces on 0.01mm"
