File: MeshHat.kicad_pcb (KiCad board)
At the start: 4 copper layers, 65 x 56.5 mm, 34 parts, among them J1 RPi_GPIO, J2 USB_B_Mini, SW1 SW_SPST, SW2 SW_SPST, U3 CAT24C128, U5 RP2040, U6 W25Q128JVS, U7 E22-900M30S, Y1 ABM8-272-T3

Commit message: WIP
Parts:
- J2: footprint Connector_USB:USB_Micro-B_XKB_U254-051T-4BH83-F1S -> Connector_USB:USB_Mini-B_Tensility_54-00023_Vertical
- U7: value E22-900M30S -> E22P-900M30S
Connections:
- J2 pad SH: (no net) -> GND

Commit message: WIP
Parts:
- added J3: Conn_01x03_Socket, Connector_JST:JST_SH_BM03B-SRSS-TB_1x03-1MP_P1.00mm_Vertical, B.Cu at (186.8, 62.0)
- added R8: 0, Resistor_SMD:R_0603_1608Metric, F.Cu at (191.5, 83.2)
- added R9: 0, Resistor_SMD:R_0603_1608Metric, F.Cu at (191.5, 85.0)
- U7: value E22P-900M30S -> E22-900M30S
- moved J2 1.83 mm to (212.5, 64.4), turned to -90 degrees
Connections:
- U5 pad 15: R_RX -> Net-(U5-GPIO12)
- U5 pad 16: R_TX -> Net-(U5-GPIO13)
Routing:
- net Net-(U5-GPIO13): track 0.00 -> 3.93 mm
- net Net-(U5-GPIO12): track 0.00 -> 1.93 mm
- net /MeshRF/~{F_SS}: track 21.4 -> 20.2 mm
- net /MeshRF/F_SD2: track 17.5 -> 16.7 mm
- net R_SWDIO: track 37.1 -> 37.8 mm
- net /E_WP: track 15.2 -> 14.6 mm
- net /MeshRF/F_SD1: track 18.4 -> 18.9 mm
- net +3.3V: track 36.4 -> 36.6 mm, vias 11 -> 10

Commit message: finish off PCB, prep for review
Parts:
- added REF**: OSHW-Logo2_14.6x12mm_SilkScreen, Symbol:OSHW-Logo2_14.6x12mm_SilkScreen, B.Cu at (208.5, 95.8)
- J2: footprint Connector_USB:USB_Mini-B_Tensility_54-00023_Vertical -> Connector_USB:USB_Mini-B_AdamTech_MUSB-B5-S-VT-TSMT-1_SMD_Vertical
- moved J2 4.63 mm to (212.4, 69.0), turned to 0 degrees
- moved U6 2.30 mm to (188.0, 61.8)
- moved R6 2.01 mm to (197.5, 71.2)
- moved R5 1.96 mm to (199.2, 71.2)
- moved C12 1.90 mm to (194.0, 69.0)
- moved C15 1.90 mm to (195.8, 69.0)
- moved C6 1.89 mm to (192.2, 68.5)
- moved C17 1.60 mm to (181.5, 68.5)
- moved C18 1.40 mm to (181.5, 66.5)
- moved C13 0.50 mm to (195.8, 61.2)
- moved C16 0.50 mm to (197.5, 61.2)
Routing:
- net /MeshRF/R_USB_DP: track 0.00 -> 14.2 mm
- net /MeshRF/R_USB_DM: track 0.00 -> 12.5 mm
- net GND: track 41.8 -> 48.5 mm, vias 35 -> 39
- net +3.3V: track 36.6 -> 39.8 mm, vias 10 -> 12
- net /MeshRF/F_SD2: track 16.7 -> 19.6 mm
- net +5V: track 34.9 -> 37.4 mm
- net /MeshRF/F_SD1: track 18.9 -> 21.1 mm
- net /MeshRF/~{F_SS}: track 20.2 -> 22.4 mm
- net /MeshRF/F_SD0: track 12.9 -> 14.4 mm
- net Net-(U5-USB_DP): track 4.37 -> 2.94 mm
- net Net-(U5-USB_DM): track 4.77 -> 3.50 mm
- net +1V1: track 25.9 -> 27.0 mm
- net /MeshRF/~{F_CLK}: track 16.1 -> 17.1 mm
- net /MeshRF/F_SD3: track 17.5 -> 18.5 mm
Other:
- board text added: "BOOT"
- board text added: "MESHHAT"
- board text added: "RST"
- board text added: "Rev A"
- board text added: "SWD"
