File: untitled.kicad_sch (KiCad schematic)
At the start: 29 parts, among them J2 USB_B_Mini, SW1 SW_SPST, SW2 SW_SPST, U5 RP2040, U6 W25Q128JVS, U7 E22-900M30S, Y1 ABM8-272-T3

Commit message: re-route the swdio lines
Parts:
- J2: footprint Connector_USB:USB_Mini-B_Lumberg_2486_01_Horizontal -> Connector_USB:USB_Mini-B_Tensility_54-00023_Vertical
Connections:
- no-connect marks 39 -> 32

Commit message: WIP
Parts:
- added J3: Conn_01x03_Socket, Connector_JST:JST_SH_BM03B-SRSS-TB_1x03-1MP_P1.00mm_Vertical, symbol Connector:Conn_01x03_Socket
Connections:
- net GND: now also J2.SH (Shield); no longer J2.6 (Shield)
- no-connect marks 32 -> 22
Changed lines of the file:
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@@
 	)
 	(no_connect
-		(at 201.93 54.61)
-	)
-	(no_connect
 		(at 82.55 27.94)
 	)
@@
 	)
 	(no_connect
-		(at 201.93 46.99)
-	)
-	(no_connect
 		(at 193.04 100.33)
 	)
@@
 	)
 	(no_connect
-		(at 201.93 36.83)
-	)
-	(no_connect
-		(at 201.93 34.29)
-	)
-	(no_connect
 		(at 193.04 72.39)
 	)
@@
 	)
 	(no_connect
-		(at 201.93 52.07)
-	)
-	(no_connect
 		(at 53.34 60.96)
 	)
@@
 	)
 	(no_connect
-		(at 201.93 39.37)
-	)
-	(no_connect
 		(at 82.55 38.1)
 	)
 	(no_connect
-		(at 201.93 57.15)
-	)
-	(no_connect
-		(at 201.93 49.53)
-	)
-	(no_connect
-		(at 201.93 41.91)
-	)
-	(no_connect
 		(at 193.04 80.01)
 	)
@@
 	)
 	(no_connect
-		(at 201.93 44.45)
-	)
-	(no_connect
 		(at 193.04 87.63)
 	)
@@
 	)
 	(label "RF_SCK"
-		(at 193.04 46.99 0)
+		(at 201.93 46.99 180)
 		(effects
 			(font
 				(size 1.27 1.27)
 			)
-			(justify left bottom)
+			(justify right bottom)
 		)
 	)
 	(label "RF_MOSI"
-		(at 193.04 49.53 0)
+		(at 201.93 49.53 180)
 		(effects
 			(font
 				(size 1.27 1.27)
 			)
-			(justify left bottom)
+			(justify right bottom)
 		)
 	)
@@
 	)
 	(label "~{RF_RST}"
-		(at 193.04 39.37 0)
+		(at 201.93 39.37 180)
 		(effects
 			(font
 				(size 1.27 1.27)
 			)
-			(justify left bottom)
+			(justify right bottom)
 		)
 	)
@@
 	)
 	(label "RF_TXEN"
-		(at 193.04 54.61 0)
+		(at 201.93 54.61 180)
 		(effects
 			(font
 				(size 1.27 1.27)
 			)
-			(justify left bottom)
+			(justify right bottom)
 		)
 	)
@@
 	)
 	(label "RF_BUSY"
-		(at 193.04 36.83 0)
+		(at 201.93 36.83 180)
 		(effects
 			(font
 				(size 1.27 1.27)
 			)
-			(justify left bottom)
+			(justify right bottom)
 		)
 	)
@@
 	)
 	(label "RF_MISO"
-		(at 193.04 41.91 0)
+		(at 201.93 41.91 180)
 		(effects
 			(font
 				(size 1.27 1.27)
 			)
-			(justify left bottom)
+			(justify right bottom)
 		)
 	)
@@
 	)
 	(label "RF_DIO2"
-		(at 193.04 52.07 0)
+		(at 201.93 52.07 180)
 		(effects
 			(font
 				(size 1.27 1.27)
 			)
-			(justify left bottom)
+			(justify right bottom)
 		)
 	)
 	(label "RF_NSS"
-		(at 193.04 44.45 0)
+		(at 201.93 44.45 180)
 		(effects
 			(font
 				(size 1.27 1.27)
 			)
-			(justify left bottom)
+			(justify right bottom)
 		)
 	)
@@
 	)
 	(label "RF_DIO1"
-		(at 193.04 34.29 0)
+		(at 201.93 34.29 180)
 		(effects
 			(font
 				(size 1.27 1.27)
 			)
-			(justify left bottom)
+			(justify right bottom)
 		)
 	)
@@
 	)
 	(label "RF_RXEN"
-		(at 193.04 57.15 0)
+		(at 201.93 57.15 180)
 		(effects
 			(font
 				(size 1.27 1.27)
 			)
-			(justify left bottom)
+			(justify right bottom)
 		)
 	)
@@
 		(pin "4"
 		)
-		(pin "6"
+		(pin "SH"
 		)
 		(pin "5"
@@
 					(unit 1)
 				)
+			)
+		)
+	)
+	(symbol
+		(lib_id "Connector:Conn_01x03_Socket")
+		(at 247.65 102.87 0)
+		(unit 1)
+		(body_style 1)
+		(exclude_from_sim no)
+		(in_bom yes)
+		(on_board yes)
+		(in_pos_files yes)
+		(dnp no)
+		(fields_autoplaced yes)
+		(property "Reference" "J3"
+			(at 248.92 101.5999 0)
+			(show_name no)
+			(do_not_autoplace no)
+			(effects
+				(font
+					(size 1.27 1.27)
+				)
+				(justify left)
+			)
+		)
+		(property "Value" "Conn_01x03_Socket"
+			(at 248.92 104.1399 0)
+			(show_name no)
+			(do_not_autoplace no)
+			(effects
+				(font
+					(size 1.27 1.27)
+				)
+				(justify left)
+			)
+		)
+		(property "Footprint" "Connector_JST:JST_SH_BM03B-SRSS-TB_1x03-1MP_P1.00mm_Vertical"
+			(at 247.65 102.87 0)
+			(hide yes)
+			(show_name no)
+			(do_not_autoplace no)
+			(effects
+				(font
+					(size 1.27 1.27)
+				)
+			)
+		)
+		(property "Datasheet" ""
+			(at 247.65 102.87 0)
+			(hide yes)
+			(show_name no)
+			(do_not_autoplace no)
+			(effects
+				(font
+					(size 1.27 1.27)
+				)
+			)
+		)
+		(property "Description" "Generic connector, single row, 01x03, script generated"
+			(at 247.65 102.87 0)
+			(hide yes)
+			(show_name no)
+			(do_not_autoplace no)
+			(effects
+				(font
+					(size 1.27 1.27)
+				)
+			)
+		)
+		(pin "2"
+		)
+		(pin "3"
+		)
+		(pin "1"
+		)
+		(instances
+			(project "MeshHat"
+				(path "/ac5b0951-7b7b-41d2-b78c-2a2e4b31a9ff/f071743a-4e4f-466f-b4e9-a324f1150a8f"
+					(reference "J3")
+					(unit 1)
+				)

Commit message: WIP
Parts:
- added R8, R9: 0, Resistor_SMD:R_0603_1608Metric, symbol Device:R_US
Connections:
- net GND: now also J3.2 (Pin_2)
- net R_RX: now also R8.2; no longer U5.15 (GPIO12)
- net R_SWCLK: now also J3.3 (Pin_3)
- net R_SWDIO: now also J3.1 (Pin_1)
- net R_TX: now also R9.2; no longer U5.16 (GPIO13)
- new net: R8.1, U5.15 (GPIO12)
- new net: R9.1, U5.16 (GPIO13)
Other:
- note added: "Resistors have to be 0.1%"

Commit message: finish off PCB, prep for review
Parts:
- J2: footprint Connector_USB:USB_Mini-B_Tensility_54-00023_Vertical -> Connector_USB:USB_Mini-B_AdamTech_MUSB-B5-S-VT-TSMT-1_SMD_Vertical
- J3: now not fitted; now left out of the parts list
Changed lines of the file:
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@@
 	(wire
 		(pts
-			(xy 240.03 105.41) (xy 242.57 105.41)
+			(xy 213.36 85.09) (xy 215.9 85.09)
 		)
 		(stroke
@@
 	(wire
 		(pts
-			(xy 240.03 100.33) (xy 242.57 100.33)
+			(xy 213.36 80.01) (xy 215.9 80.01)
 		)
 		(stroke
@@
 	(wire
 		(pts
-			(xy 240.03 102.87) (xy 242.57 102.87)
+			(xy 213.36 82.55) (xy 215.9 82.55)
 		)
 		(stroke
@@
 	(global_label "R_SWCLK"
 		(shape input)
-		(at 240.03 105.41 180)
+		(at 213.36 85.09 180)
 		(fields_autoplaced yes)
 		(effects
@@
 		)
 		(property "Intersheetrefs" "${INTERSHEET_REFS}"
-			(at 228.5782 105.41 0)
+			(at 201.9082 85.09 0)
 			(hide yes)
 			(show_name no)
@@
 	(global_label "R_SWDIO"
 		(shape input)
-		(at 240.03 100.33 180)
+		(at 213.36 80.01 180)
 		(fields_autoplaced yes)
 		(effects
@@
 		)
 		(property "Intersheetrefs" "${INTERSHEET_REFS}"
-			(at 228.941 100.33 0)
+			(at 202.271 80.01 0)
 			(hide yes)
 			(show_name no)
@@
 			)
 		)
-		(property "Footprint" "Connector_USB:USB_Mini-B_Tensility_54-00023_Vertical"
+		(property "Footprint" "Connector_USB:USB_Mini-B_AdamTech_MUSB-B5-S-VT-TSMT-1_SMD_Vertical"
 			(at 78.74 34.29 0)
 			(hide yes)
@@
 	(symbol
 		(lib_id "power:GND")
-		(at 240.03 102.87 270)
+		(at 213.36 82.55 270)
 		(unit 1)
 		(body_style 1)
@@
 		(fields_autoplaced yes)
 		(property "Reference" "#PWR013"
-			(at 233.68 102.87 0)
+			(at 207.01 82.55 0)
 			(hide yes)
 			(show_name no)
@@
 		)
 		(property "Value" "GND"
-			(at 236.22 102.8699 90)
+			(at 209.55 82.5499 90)
 			(show_name no)
 			(do_not_autoplace no)
@@
 		)
 		(property "Footprint" ""
-			(at 240.03 102.87 0)
+			(at 213.36 82.55 0)
 			(hide yes)
 			(show_name no)
@@
 		)
 		(property "Datasheet" ""
-			(at 240.03 102.87 0)
+			(at 213.36 82.55 0)
 			(hide yes)
 			(show_name no)
@@
 		)
 		(property "Description" "Power symbol creates a global label with name \"GND\" , ground"
-			(at 240.03 102.87 0)
+			(at 213.36 82.55 0)
 			(hide yes)
 			(show_name no)
@@
 	(symbol
 		(lib_id "Connector:Conn_01x03_Socket")
-		(at 247.65 102.87 0)
+		(at 220.98 82.55 0)
 		(unit 1)
 		(body_style 1)
 		(exclude_from_sim no)
-		(in_bom yes)
+		(in_bom no)
 		(on_board yes)
 		(in_pos_files yes)
-		(dnp no)
+		(dnp yes)
 		(property "Reference" "J3"
-			(at 228.854 97.282 0)
+			(at 202.184 76.962 0)
 			(show_name no)
 			(do_not_autoplace no)
@@
 		)
 		(property "Value" "Conn_01x03_Socket"
-			(at 228.854 108.458 0)
+			(at 202.184 88.138 0)
 			(show_name no)
 			(do_not_autoplace no)
@@
 		)
 		(property "Footprint" "Connector_JST:JST_SH_BM03B-SRSS-TB_1x03-1MP_P1.00mm_Vertical"
-			(at 247.65 102.87 0)
+			(at 220.98 82.55 0)
 			(hide yes)
 			(show_name no)
@@
 		)
 		(property "Datasheet" ""
-			(at 247.65 102.87 0)
+			(at 220.98 82.55 0)
 			(hide yes)
 			(show_name no)
@@
 		)
 		(property "Description" "Generic connector, single row, 01x03, script generated"
-			(at 247.65 102.87 0)
+			(at 220.98 82.55 0)
 			(hide yes)
 			(show_name no)
